File: hardware/developmentboard.kicad_sch (KiCad schematic)
At the start: 12 parts, among them J1 Conn_01x03_Female, J2 Conn_01x04_Female, J3 Conn_01x03_Female, J4 Conn_01x04_Female, J5 Conn_01x11_Male, U1 ADS7960, U2 DRV5053VAQDBZR

Commit message: ??? made a board lol
Parts:
- U2: footprint Package_TO_SOT_SMD:SOT-23-5_HandSoldering -> Package_TO_SOT_SMD:SOT-23
Connections:
- net VA renamed +3V3
