File: hardware/developmentboard.kicad_pcb (KiCad board)
At the start: 2 copper layers, 12 parts, among them J1 Conn_01x03_Female, J2 Conn_01x04_Female, J3 Conn_01x03_Female, J4 Conn_01x04_Female, J5 Conn_01x11_Male, U1 ADS7960, U2 DRV5053VAQDBZR

Commit message: ??? made a board lol
Parts:
- C2, C5: moved to B.Cu
- U2: footprint Package_TO_SOT_SMD:SOT-23-5_HandSoldering -> Package_TO_SOT_SMD:SOT-23
- moved J5 68.6 mm to (160.4, 66.1), turned to 90 degrees
- moved C4 41.2 mm to (142.4, 85.5)
- moved U2 36.9 mm to (101.6, 96.0)
- moved J4 30.0 mm to (90.8, 76.1)
- moved C5 29.4 mm to (132.5, 84.8), turned to 180 degrees
- moved J1 26.2 mm to (90.9, 65.5)
- moved U1 21.7 mm to (140.0, 78.0), turned to 90 degrees
- moved J3 20.6 mm to (110.4, 65.3), turned to 90 degrees
- moved C1 16.4 mm to (136.6, 85.1)
- moved C2 13.2 mm to (136.2, 71.2), turned to 180 degrees
- moved C3 8.84 mm to (104.4, 90.9)
- moved J2 6.17 mm to (136.5, 65.7), turned to 90 degrees

Commit message: added 2.5v regulator and 12 keys
added 2.5v regulator and 12 keys

added 2.5v regulator and 12 keys
Parts:
- added C10: C_Small, Capacitor_THT:CP_Radial_D4.0mm_P1.50mm, F.Cu at (160.2, 95.0)
- added C11: C_Small, Capacitor_THT:CP_Radial_D4.0mm_P1.50mm, F.Cu at (165.8, 95.0)
- added C12: C_Small, Capacitor_THT:CP_Radial_D4.0mm_P1.50mm, F.Cu at (171.4, 83.9)
- added C13: C_Small, Capacitor_THT:CP_Radial_D4.0mm_P1.50mm, F.Cu at (160.2, 89.4)
- added C14: C_Small, Capacitor_THT:CP_Radial_D4.0mm_P1.50mm, F.Cu at (165.8, 83.9)
- added C15: C_Small, Capacitor_THT:CP_Radial_D4.0mm_P1.50mm, F.Cu at (171.4, 89.4)
- added C16: C_Small, Capacitor_THT:CP_Radial_D4.0mm_P1.50mm, F.Cu at (154.6, 95.0)
- added C6: C_Small, Capacitor_THT:CP_Radial_D4.0mm_P1.50mm, F.Cu at (165.8, 89.4)
- added C7: C_Small, Capacitor_THT:CP_Radial_D4.0mm_P1.50mm, F.Cu at (154.6, 83.9)
- added C8: C_Small, Capacitor_THT:CP_Radial_D4.0mm_P1.50mm, F.Cu at (160.2, 83.9)
- added C9: C_Small, Capacitor_THT:CP_Radial_D4.0mm_P1.50mm, F.Cu at (154.6, 89.4)
- added U10: DRV5055A1xDBZxQ1, Package_TO_SOT_SMD:SOT-23, F.Cu at (177.4, 87.8)
- added U11: DRV5055A1xDBZxQ1, Package_TO_SOT_SMD:SOT-23, F.Cu at (177.4, 83.3)
- added U12: DRV5055A1xDBZxQ1, Package_TO_SOT_SMD:SOT-23, F.Cu at (155.0, 100.0)
- added U13: DRV5055A1xDBZxQ1, Package_TO_SOT_SMD:SOT-23, F.Cu at (177.4, 92.2)
- added U14: AP2138N-2.5TRG1, Package_TO_SOT_SMD:SOT-23, F.Cu at (149.2, 72.8)
- added U2: DRV5055A1xDBZxQ1, Package_TO_SOT_SMD:SOT-23, F.Cu at (164.7, 100.0)
- added U3: DRV5055A1xDBZxQ1, Package_TO_SOT_SMD:SOT-23, F.Cu at (159.8, 100.0)
- added U4: DRV5055A1xDBZxQ1, Package_TO_SOT_SMD:SOT-23, F.Cu at (182.2, 87.8)
- added U5: DRV5055A1xDBZxQ1, Package_TO_SOT_SMD:SOT-23, F.Cu at (176.6, 96.7)
- added U6: DRV5055A1xDBZxQ1, Package_TO_SOT_SMD:SOT-23, F.Cu at (182.2, 83.3)
- added U7: DRV5055A1xDBZxQ1, Package_TO_SOT_SMD:SOT-23, F.Cu at (169.6, 100.0)
- added U8: DRV5055A1xDBZxQ1, Package_TO_SOT_SMD:SOT-23, F.Cu at (187.1, 83.3)
- added U9: DRV5055A1xDBZxQ1, Package_TO_SOT_SMD:SOT-23, F.Cu at (171.8, 94.4)
- C2, C5: moved to F.Cu
- J1: value Conn_01x03_Female -> MXO AINP; footprint Connector_PinHeader_2.54mm:PinHeader_1x03_P2.54mm_Horizontal -> Connector_PinHeader_2.54mm:PinHeader_1x02_P2.54mm_Vertical
- J2: value Conn_01x04_Female -> SPI Header
- J3: value Conn_01x03_Female -> Power; footprint Connector_PinHeader_2.54mm:PinHeader_1x03_P2.54mm_Horizontal -> Connector_PinHeader_2.54mm:PinHeader_1x03_P2.54mm_Vertical
- J4: value Conn_01x04_Female -> GPIO
- J5: value Conn_01x11_Male -> Channel Breakout; footprint Connector_PinHeader_2.54mm:PinHeader_1x11_P2.54mm_Horizontal -> Connector_PinHeader_2.54mm:PinHeader_1x11_P2.54mm_Vertical
- moved J1 60.1 mm to (151.0, 65.7), turned to 90 degrees
- moved C3 6.02 mm to (98.7, 92.7)
- moved C2 5.02 mm to (132.2, 74.3), turned to 0 degrees
- moved C4 4.95 mm to (146.3, 82.4)
- moved C1 4.72 mm to (140.5, 82.4)
- moved U1 3.47 mm to (141.4, 74.8)
- moved C5 3.44 mm to (135.0, 82.4), turned to 0 degrees
- moved U2 3.23 mm to (98.6, 97.2)
- moved J5 1.02 mm to (160.8, 65.2)
Connections:
- C1 pad 1: Net-(J1-Pin_3) -> Vref
- U1 pad 4: Net-(J1-Pin_3) -> Vref
- U1 pad 7: Net-(J1-Pin_2) -> Net-(J1-Pin_1)
- U1 pad 8: Net-(J1-Pin_1) -> Net-(J1-Pin_2)
Routing:
- net Net-(J2-Pin_4): track 0.00 -> 8.98 mm
- net Net-(J2-Pin_1): track 0.00 -> 7.54 mm
- net Net-(J2-Pin_3): track 0.00 -> 7.31 mm
- net Net-(J2-Pin_2): track 0.00 -> 6.40 mm
